File: Kicad-CheeseCake-SlimeTrackers(edit).kicad_sch (KiCad schematic)
At the start: 15 parts, among them J2 USB_C-16p, Q1 UMH3N, SW1 SW_SPDT, U2 TP4057, U3 CH340K

Commit message: updt
Parts:
- added C3: 100nF, symbol Device:C_Small_US
- added C4: 1uF, symbol Device:C_Small_US
- added ESP1: ~, symbol _symbolsslime:ESP12F_edit
- added R5: 4.7k, symbol Device:R
Connections:
- net +3V3: now also C3.1, C4.1, ESP1.8 (VCC)
- net GND: now also C3.2, C4.2, ESP1.9 (GND), R5.2
- net GPIO0: now also ESP1.12 (GPIO0)
- net RST: now also ESP1.1 (RST)
- net RX: now also ESP1.15 (RXD0)
- net TX: now also ESP1.16 (TXD0)
- new net ADC: ESP1.2 (ADC)
- new net EN: ESP1.3 (EN)
- new net GPIO15: ESP1.10 (GPIO15), R5.1
- new net LED: ESP1.11 (GPIO2)
- new net SCL: ESP1.14 (GPIO5)
- new net SDA: ESP1.13 (GPIO4)
- no-connect marks 5 -> 15

Commit message: updt
Parts:
- added R10, R6, R7, R8, R9: 4.7k, symbol Device:R
Connections:
- net +3V3: now also R10.2, R6.2, R7.2, R8.2, R9.2
- net EN: now also R6.1
- net GPIO0: now also R8.1
- net RST: now also R7.1
- net SCL: now also R10.1
- net SDA: now also R9.1
Other:
- moved on the sheet: R5

Commit message: updt
Parts:
- removed C2: 100nF, symbol Device:C
- added C2: 100nF, symbol Device:C_Small_US
- U3: footprint Package_SO:SSOP-10-1EP_3.9x4.9mm_P1mm_EP2.1x3.3mm -> (none)
Connections:
- net +3V3: now also C2.1
- net GND: now also C2.2

Commit message: updt
Parts:
- added C5, C6: 1uF, symbol Device:C_Small_US
- added U4: ME6211C33M5, Package_TO_SOT_SMD:SOT-23-5, symbol Regulator_Linear:ME6211C33M5
Connections:
- net +3V3: now also C6.1, U4.5 (V_{OUT})
- net GND: now also C5.2, C6.2, U4.2 (V_{SS})
- net VIN: now also C5.1, U4.1 (V_{IN}), U4.3 (CE)
Other:
- note added: "LDO3V3 ME6211C33M5G-N"

Commit message: updt
Parts:
- added C7, C8: 100nF, symbol Device:C_Small_US
- added J3: 4P4C, symbol Connector:4P4C
- U1: value ~ -> ICM-45686
Connections:
- net +3V3: now also U1.2 (+3V3), C7.1, C8.1, J3.1; no longer C2.1, U3.10 (V3)
- net GND: now also U1.3 (GND), C7.2, C8.2, J3.2
- net SCL: now also U1.4 (SCL), J3.3
- net SDA: now also U1.5 (SDA), J3.4
- new net: C2.1, U3.10 (V3)
- no-connect marks 15 -> 24
Other:
- note added: "AUX JST CON"
- note added: "Taken from Sorakage's design, re implemented in kidkad for personal slimes"
- note added: "UNTESTED"
- moved on the sheet: U1, U3

Commit message: inital footprint assignment
erc tests passed
some potential issues regarding +3v3 flag - cleared tests for now

some footprints could be wrong and are placeholder
Parts:
- B1, J1: footprint (none) -> Connector_PinHeader_2.54mm:PinHeader_1x02_P2.54mm_Horizontal
- C1, C2, C3, C4, C5, C6, C7, C8: footprint (none) -> Capacitor_SMD:C_0603_1608Metric
- ESP1: footprint (none) -> SlimeFootprints:ESP12F-Devkit-V3
- J2: footprint (none) -> Connector_USB:USB_C_Receptacle_HCTL_HC-TYPE-C-16P-01A
- J3: footprint (none) -> Connector_Hirose:Hirose_DF13C_CL535-0405-0-51_1x05-1MP_P1.25mm_Vertical
- L1: footprint (none) -> LED_SMD:LED_RGB_Cree-PLCC-6_6x5mm_P2.1mm
- Q1: footprint (none) -> Package_TO_SOT_SMD:SOT-363_SC-70-6
- R1, R10, R2, R3, R4, R5, R6, R7, R8, R9: footprint (none) -> Resistor_SMD:R_0603_1608Metric
- SW1: footprint (none) -> SlimeFootprints:SW_SSSS811101
- U1: footprint (none) -> Package_LGA:Bosch_LGA-14_3x2.5mm_P0.5mm
- U3: footprint (none) -> Package_SO:SOIC-10_3.9x4.9mm_P1mm
Changed lines of the file:
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@@
 			)
 		)
-		(property "Footprint" ""
+		(property "Footprint" "Resistor_SMD:R_0603_1608Metric"
 			(at 49.53 185.928 90)
 			(effects
@@
 			)
 		)
-		(property "Footprint" ""
+		(property "Footprint" "Resistor_SMD:R_0603_1608Metric"
 			(at 49.53 182.118 90)
 			(effects
@@
 			)
 		)
-		(property "Footprint" ""
+		(property "Footprint" "Resistor_SMD:R_0603_1608Metric"
 			(at 22.352 39.37 90)
 			(effects
@@
 			)
 		)
-		(property "Footprint" ""
+		(property "Footprint" "Package_LGA:Bosch_LGA-14_3x2.5mm_P0.5mm"
 			(at 128.27 144.78 0)
 			(effects
@@
 			)
 		)
-		(property "Footprint" ""
+		(property "Footprint" "Connector_Hirose:Hirose_DF13C_CL535-0405-0-51_1x05-1MP_P1.25mm_Vertical"
 			(at 144.78 96.52 90)
 			(effects
@@
 			)
 		)
-		(property "Footprint" ""
+		(property "Footprint" "Capacitor_SMD:C_0603_1608Metric"
 			(at 19.05 160.02 0)
 			(effects
@@
 			)
 		)
-		(property "Footprint" ""
+		(property "Footprint" "Capacitor_SMD:C_0603_1608Metric"
 			(at 86.36 102.87 0)
 			(effects
@@
 			)
 		)
-		(property "Footprint" ""
+		(property "Footprint" "Capacitor_SMD:C_0603_1608Metric"
 			(at 78.74 102.87 0)
 			(effects
@@
 			)
 		)
-		(property "Footprint" ""
+		(property "Footprint" "SlimeFootprints:ESP12F-Devkit-V3"
 			(at 43.18 156.21 0)
 			(effects
@@
 			)
 		)
-		(property "Footprint" ""
+		(property "Footprint" "Capacitor_SMD:C_0603_1608Metric"
 			(at 99.06 147.32 0)
 			(effects
@@
 			)
 		)
-		(property "Footprint" ""
+		(property "Footprint" "LED_SMD:LED_RGB_Cree-PLCC-6_6x5mm_P2.1mm"
 			(at 130.81 54.61 0)
 			(effects
@@
 			)
 		)
-		(property "Footprint" ""
+		(property "Footprint" "Connector_PinHeader_2.54mm:PinHeader_1x02_P2.54mm_Horizontal"
 			(at 148.59 53.34 0)
 			(effects
@@
 			)
 		)
-		(property "Footprint" ""
+		(property "Footprint" "Resistor_SMD:R_0603_1608Metric"
 			(at 24.892 58.42 90)
 			(effects
@@
 			)
 		)
-		(property "Footprint" ""
+		(property "Footprint" "Capacitor_SMD:C_0603_1608Metric"
 			(at 36.83 77.47 0)
 			(effects
@@
 			)
 		)
-		(property "Footprint" ""
+		(property "Footprint" "Package_SO:SOIC-10_3.9x4.9mm_P1mm"
 			(at 31.75 113.03 0)
 			(effects
@@
 			)
 		)
-		(property "Footprint" ""
+		(property "Footprint" "Resistor_SMD:R_0603_1608Metric"
 			(at 95.25 44.958 90)
 			(effects
@@
 			)
 		)
-		(property "Footprint" ""
+		(property "Footprint" "Resistor_SMD:R_0603_1608Metric"
 			(at 26.67 180.848 90)
 			(effects
@@
 			)
 		)
-		(property "Footprint" ""
+		(property "Footprint" "Resistor_SMD:R_0603_1608Metric"
 			(at 144.78 28.702 90)
 			(effects
@@
 			)
 		)
-		(property "Footprint" ""
+		(property "Footprint" "Resistor_SMD:R_0603_1608Metric"
 			(at 49.53 193.548 90)
 			(effects
@@
 			)
 		)
-		(property "Footprint" ""
+		(property "Footprint" "Capacitor_SMD:C_0603_1608Metric"
 			(at 105.41 147.32 0)
 			(effects
@@
 			)
 		)
-		(property "Footprint" ""
+		(property "Footprint" "Connector_PinHeader_2.54mm:PinHeader_1x02_P2.54mm_Horizontal"
 			(at 97.79 53.34 0)
 			(effects
@@
 			)
 		)
-		(property "Footprint" ""
+		(property "Footprint" "Capacitor_SMD:C_0603_1608Metric"
 			(at 149.86 24.4348 0)
 			(effects
@@
 			)
 		)
-		(property "Footprint" ""
+		(property "Footprint" "SlimeFootprints:SW_SSSS811101"
 			(at 95.25 27.94 0)
 			(effects
@@
 			)
 		)
-		(property "Footprint" ""
+		(property "Footprint" "Package_TO_SOT_SMD:SOT-363_SC-70-6"
 			(at 55.88 96.52 0)
 			(effects
@@
 			)
 		)
-		(property "Footprint" ""
+		(property "Footprint" "Resistor_SMD:R_0603_1608Metric"
 			(at 49.53 189.738 90)
 			(effects
@@
 			)
 		)
-		(property "Footprint" ""
+		(property "Footprint" "Connector_USB:USB_C_Receptacle_HCTL_HC-TYPE-C-16P-01A"
 			(at 55.88 39.37 0)
 			(effects
@@
 			)
 		)
-		(property "Footprint" ""
+		(property "Footprint" "Resistor_SMD:R_0603_1608Metric"
 			(at 49.53 178.308 90)
 			(effects
@@
 			)
 		)
-		(property "Footprint" ""
+		(property "Footprint" "Capacitor_SMD:C_0603_1608Metric"
 			(at 22.86 160.02 0)
 			(effects

Commit message: started pcb
pcb inital
Parts:
- added BT1: battery, symbol Device:Battery_Cell
- B1, J1: footprint Connector_PinHeader_2.54mm:PinHeader_1x02_P2.54mm_Horizontal -> Connector_PinSocket_2.54mm:PinSocket_1x02_P2.54mm_Vertical
- ESP1: footprint SlimeFootprints:ESP12F-Devkit-V3 -> (none)
- U1: footprint Package_LGA:Bosch_LGA-14_3x2.5mm_P0.5mm -> Connector_PinHeader_1.00mm:PinHeader_1x07_P1.00mm_Vertical
Connections:
- net BAT+ is gone; now on net +5V: B1.1, C1.1, R3.1, SW1.1 (A), U2.3 (BAT)
- net +5V: now also BT1.1 (+)
- net GND: now also BT1.2 (-)

Commit message: updt
lots of fixes to footprints
Parts:
- ESP1: footprint (none) -> SlimeFootprints:ESP-12F
- L1: footprint LED_SMD:LED_RGB_Cree-PLCC-6_6x5mm_P2.1mm -> SlimeFootprints:LED_CLMVC-FKA-CG1H1A1BB7D3C3
Changed lines of the file:
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@@
 			)
 		)
-		(property "Footprint" ""
+		(property "Footprint" "SlimeFootprints:ESP-12F"
 			(at 43.18 156.21 0)
 			(effects
@@
 			)
 		)
-		(property "Footprint" "LED_SMD:LED_RGB_Cree-PLCC-6_6x5mm_P2.1mm"
+		(property "Footprint" "SlimeFootprints:LED_CLMVC-FKA-CG1H1A1BB7D3C3"
 			(at 130.81 54.61 0)
 			(effects
