File: Kicad-CheeseCake-SlimeTrackers(edit).kicad_sch (KiCad schematic)
At the start: 31 parts, among them J2 USB_C-16p, J3 4P4C, Q1 UMH3N, SW1 SW_SPDT, U1 ICM-45686, U2 TP4057, U3 CH340K, U4 ME6211C33M5

Commit message: fixes
board will be 33x35 or bigger
Parts:
- removed BT1: battery, symbol Device:Battery_Cell
- J1: now left out of the parts list
- U1: footprint Connector_PinHeader_1.00mm:PinHeader_1x07_P1.00mm_Vertical -> Connector_PinHeader_2.54mm:PinHeader_1x07_P2.54mm_Vertical
Connections:
- net +5V: no longer B1.1, C1.1, R3.1, SW1.1 (A), U2.3 (BAT)
- new net BAT+: B1.1, C1.1, R3.1, SW1.1 (A), U2.3 (BAT)
Changed lines of the file:
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@@
 	(text_box "pwr flags"
 		(exclude_from_sim no)
-		(at 175.956 64.8238 0)
+		(at 173.99 36.83 0)
 		(size 11.43 3.81)
 		(margins 0.9525 0.9525 0.9525 0.9525)
@@
 	)
 	(junction
-		(at 182.88 40.64)
-		(diameter 0)
-		(color 0 0 0 0)
-	)
-	(junction
 		(at 22.86 156.21)
 		(diameter 0)
@@
 	(wire
 		(pts
-			(xy 176.53 40.64) (xy 182.88 40.64)
-		)
-		(stroke
-			(width 0)
-			(type default)
-		)
-	)
-	(wire
-		(pts
 			(xy 87.63 93.98) (xy 88.9 93.98)
 		)
@@
 		)
 	)
-	(global_label "BAT+"
-		(shape input)
-		(at 176.53 40.64 90)
-		(fields_autoplaced yes)
-		(effects
-			(font
-				(size 1.27 1.27)
-				(thickness 0.254)
-				(bold yes)
-			)
-			(justify left)
-		)
-		(property "Intersheetrefs" "${INTERSHEET_REFS}"
-			(at 176.53 32.2802 90)
-			(effects
-				(font
-					(size 1.27 1.27)
-				)
-				(justify left)
-				(hide yes)
-			)
-		)
-	)
 	(global_label "DN"
 		(shape input)
@@
 			)
 		)
-		(property "Footprint" "Connector_PinHeader_1.00mm:PinHeader_1x07_P1.00mm_Vertical"
+		(property "Footprint" "Connector_PinHeader_2.54mm:PinHeader_1x07_P2.54mm_Vertical"
 			(at 128.27 144.78 0)
 			(effects
@@
 	)
 	(symbol
-		(lib_id "Device:Battery_Cell")
-		(at 182.88 45.72 0)
-		(unit 1)
-		(exclude_from_sim no)
-		(in_bom no)
-		(on_board no)
-		(dnp no)
-		(fields_autoplaced yes)
-		(property "Reference" "BT1"
-			(at 186.69 42.6084 0)
-			(effects
-				(font
-					(size 1.27 1.27)
-				)
-				(justify left)
-			)
-		)
-		(property "Value" "battery"
-			(at 186.69 45.1484 0)
-			(effects
-				(font
-					(size 1.27 1.27)
-				)
-				(justify left)
-			)
-		)
-		(property "Footprint" ""
-			(at 182.88 44.196 90)
-			(effects
-				(font
-					(size 1.27 1.27)
-				)
-				(hide yes)
-			)
-		)
-		(property "Datasheet" "~"
-			(at 182.88 44.196 90)
-			(effects
-				(font
-					(size 1.27 1.27)
-				)
-				(hide yes)
-			)
-		)
-		(property "Description" "Single-cell battery"
-			(at 182.88 45.72 0)
-			(effects
-				(font
-					(size 1.27 1.27)
-				)
-				(hide yes)
-			)
-		)
-		(pin "1"
-		)
-		(pin "2"
-		)
-		(instances
-			(project ""
-				(path "/cb0cfa68-01d6-40dd-8faf-d58d01d74d01"
-					(reference "BT1")
-					(unit 1)
-				)
-			)
-		)
-	)
-	(symbol
 		(lib_id "Device:C_Small_US")
 		(at 99.06 147.32 0)
@@
 	)
 	(symbol
-		(lib_id "power:GND")
-		(at 182.88 48.26 0)
-		(unit 1)
-		(exclude_from_sim no)
-		(in_bom yes)
-		(on_board yes)
-		(dnp no)
-		(fields_autoplaced yes)
-		(property "Reference" "#PWR033"
-			(at 182.88 54.61 0)
-			(effects
-				(font
-					(size 1.27 1.27)
-				)
-				(hide yes)
-			)
-		)
-		(property "Value" "GND"
-			(at 182.88 53.34 0)
-			(effects
-				(font
-					(size 1.27 1.27)
-				)
-			)
-		)
-		(property "Footprint" ""
-			(at 182.88 48.26 0)
-			(effects
-				(font
-					(size 1.27 1.27)
-				)
-				(hide yes)
-			)
-		)
-		(property "Datasheet" ""
-			(at 182.88 48.26 0)
-			(effects
-				(font
-					(size 1.27 1.27)
-				)
-				(hide yes)
-			)
-		)
-		(property "Description" "Power symbol creates a global label with name \"GND\" , ground"
-			(at 182.88 48.26 0)
-			(effects
-				(font
-					(size 1.27 1.27)
-				)
-				(hide yes)
-			)
-		)
-		(pin "1"
-		)
-		(instances
-			(project ""
-				(path "/cb0cfa68-01d6-40dd-8faf-d58d01d74d01"
-					(reference "#PWR033")
-					(unit 1)
-				)
-			)
-		)
-	)
-	(symbol
 		(lib_id "power:+5V")
 		(at 129.54 20.32 0)
@@
 	)
 	(symbol
-		(lib_id "power:+5V")
-		(at 182.88 40.64 0)
-		(unit 1)
-		(exclude_from_sim no)
-		(in_bom yes)
-		(on_board yes)
-		(dnp no)
-		(fields_autoplaced yes)
-		(property "Reference" "#PWR026"
-			(at 182.88 44.45 0)
-			(effects
-				(font
-					(size 1.27 1.27)
-				)
-				(hide yes)
-			)
-		)
-		(property "Value" "+5V"
-			(at 182.88 35.56 0)
-			(effects
-				(font
-					(size 1.27 1.27)
-				)
-			)
-		)
-		(property "Footprint" ""
-			(at 182.88 40.64 0)
-			(effects
-				(font
-					(size 1.27 1.27)
-				)
-				(hide yes)
-			)
-		)
-		(property "Datasheet" ""
-			(at 182.88 40.64 0)
-			(effects
-				(font
-					(size 1.27 1.27)
-				)
-				(hide yes)
-			)
-		)
-		(property "Description" "Power symbol creates a global label with name \"+5V\""
-			(at 182.88 40.64 0)
-			(effects
-				(font
-					(size 1.27 1.27)
-				)
-				(hide yes)
-			)
-		)
-		(pin "1"
-		)
-		(instances
-			(project ""
-				(path "/cb0cfa68-01d6-40dd-8faf-d58d01d74d01"
-					(reference "#PWR026")
-					(unit 1)
-				)
-			)
-		)
-	)
-	(symbol
 		(lib_id "power:GND")
 		(at 151.13 30.48 90)
@@
 		(at 97.79 53.34 0)
 		(unit 1)
-		(exclude_from_sim no)
-		(in_bom yes)
-		(on_board yes)
+		(exclude_from_sim yes)
+		(in_bom no)
+		(on_board no)
 		(dnp no)
 		(fields_autoplaced yes)

Commit message: updt
updt
Parts:
- J2: footprint Connector_USB:USB_C_Receptacle_HCTL_HC-TYPE-C-16P-01A -> KH-TYPE-C-16P:KINGHELM_KH-TYPE-C-16P; symbol Connector:USB_C_Receptacle_USB2.0_16P -> _symbolsslime:KH-TYPE-C-16P; Availability (none) -> Not in stock; Check_prices (none) -> https://www.snapeda.com/parts/KH-TYPE-C-16P/Kinghelm/view-p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; MANUFACTURER (none) -> Kinghelm; MAXIMUM_PACKAGE_HEIGHT (none) -> 3.41mm; MF (none) -> kinghelm; MP (none) -> KH-TYPE-C-16P; PARTREV (none) -> A0; Package (none) -> None; Price (none) -> None; SNAPEDA_PN (none) -> KH-TYPE-C-16P; STANDARD (none) -> Manufacturer Recommendations; SnapEDA_Link (none) -> https://www.snapeda.com/parts/KH-TYPE-C-16P/Kinghelm/view-p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
Connections:
- net +5V: no longer J2.11 (VBUS), J2.2 (VBUS)
- net DN: no longer J2.5 (DN2), J2.7 (DN1)
- net DP: no longer J2.6 (DP1), J2.8 (DP2)
- net GND: no longer J2.1 (GND), J2.12 (GND), J2.13 (SHELL), J2.14 (SHELL)
- net at R1.1: no longer J2.4 (CC1)
- net at R2.1: no longer J2.10 (CC2)
- new net: J2.A12_B1 (GND), J2.A1_B12 (GND)
- new net: J2.A4_B9 (VBUS), J2.A9_B4 (VBUS)
- new net: J2.SH1 (SHIELD), J2.SH2 (SHIELD), J2.SH3 (SHIELD), J2.SH4 (SHIELD)
- no-connect marks 24 -> 23
Changed lines of the file:
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@@
 	)
 	(junction
-		(at 67.31 46.99)
-		(diameter 0)
-		(color 0 0 0 0)
-	)
-	(junction
 		(at 105.41 139.7)
 		(diameter 0)
@@
 	)
 	(no_connect
-		(at 36.83 27.94)
-	)
-	(no_connect
 		(at 36.83 45.72)
 	)
@@
 	(wire
 		(pts
-			(xy 36.83 31.75) (xy 24.13 31.75)
-		)
-		(stroke
-			(width 0)
-			(type default)
-		)
-	)
-	(wire
-		(pts
 			(xy 31.75 161.29) (xy 30.48 161.29)
 		)
@@
 	(wire
 		(pts
-			(xy 19.05 20.32) (xy 36.83 20.32)
-		)
-		(stroke
-			(width 0)
-			(type default)
-		)
-	)
-	(wire
-		(pts
 			(xy 148.59 30.48) (xy 151.13 30.48)
 		)
@@
 	(wire
 		(pts
-			(xy 19.05 62.23) (xy 24.13 62.23)
-		)
-		(stroke
-			(width 0)
-			(type default)
-		)
-	)
-	(wire
-		(pts
 			(xy 36.83 62.23) (xy 67.31 62.23)
 		)
@@
 	(wire
 		(pts
-			(xy 33.02 24.13) (xy 36.83 24.13)
-		)
-		(stroke
-			(width 0)
-			(type default)
-		)
-	)
-	(wire
-		(pts
 			(xy 96.52 105.41) (xy 86.36 105.41)
 		)
@@
 	(wire
 		(pts
-			(xy 24.13 31.75) (xy 24.13 35.56)
-		)
-		(stroke
-			(width 0)
-			(type default)
-		)
-	)
-	(wire
-		(pts
 			(xy 88.9 88.9) (xy 81.28 88.9)
 		)
@@
 	(wire
 		(pts
-			(xy 19.05 62.23) (xy 19.05 20.32)
-		)
-		(stroke
-			(width 0)
-			(type default)
-		)
-	)
-	(wire
-		(pts
 			(xy 30.48 83.82) (xy 31.75 83.82)
 		)
@@
 	(wire
 		(pts
-			(xy 67.31 62.23) (xy 67.31 46.99)
-		)
-		(stroke
-			(width 0)
-			(type default)
-		)
-	)
-	(wire
-		(pts
 			(xy 105.41 149.86) (xy 105.41 152.4)
 		)
@@
 	(wire
 		(pts
-			(xy 67.31 29.21) (xy 67.31 46.99)
-		)
-		(stroke
-			(width 0)
-			(type default)
-		)
-	)
-	(wire
-		(pts
 			(xy 99.06 149.86) (xy 99.06 152.4)
 		)
@@
 	)
 	(symbol
-		(lib_id "power:+5V")
-		(at 33.02 24.13 90)
-		(unit 1)
-		(exclude_from_sim no)
-		(in_bom yes)
-		(on_board yes)
-		(dnp no)
-		(fields_autoplaced yes)
-		(property "Reference" "#PWR02"
-			(at 36.83 24.13 0)
-			(effects
-				(font
-					(size 1.27 1.27)
-				)
-				(hide yes)
-			)
-		)
-		(property "Value" "+5V"
-			(at 29.21 24.1299 90)
-			(effects
-				(font
-					(size 1.27 1.27)
-				)
-				(justify left)
-			)
-		)
-		(property "Footprint" ""
-			(at 33.02 24.13 0)
-			(effects
-				(font
-					(size 1.27 1.27)
-				)
-				(hide yes)
-			)
-		)
-		(property "Datasheet" ""
-			(at 33.02 24.13 0)
-			(effects
-				(font
-					(size 1.27 1.27)
-				)
-				(hide yes)
-			)
-		)
-		(property "Description" "Power symbol creates a global label with name \"+5V\""
-			(at 33.02 24.13 0)
-			(effects
-				(font
-					(size 1.27 1.27)
-				)
-				(hide yes)
-			)
-		)
-		(pin "1"
-		)
-		(instances
-			(project ""
-				(path "/cb0cfa68-01d6-40dd-8faf-d58d01d74d01"
-					(reference "#PWR02")
-					(unit 1)
-				)
-			)
-		)
-	)
-	(symbol
 		(lib_id "power:GND")
 		(at 24.13 64.77 0)
@@
 	)
 	(symbol
-		(lib_id "Connector:USB_C_Receptacle_USB2.0_16P")
-		(at 52.07 39.37 0)
+		(lib_id "_symbolsslime:KH-TYPE-C-16P")
+		(at 63.5 34.29 180)
 		(unit 1)
 		(exclude_from_sim no)
@@
 		(fields_autoplaced yes)
 		(property "Reference" "J2"
-			(at 40.64 39.3701 0)
+			(at 74.93 34.2899 0)
 			(effects
 				(font
@@
 		)
 		(property "Value" "USB_C-16p"
-			(at 52.07 16.51 0)
+			(at 63.5 19.05 0)
 			(effects
 				(font
@@
 			)
 		)
-		(property "Footprint" "Connector_USB:USB_C_Receptacle_HCTL_HC-TYPE-C-16P-01A"
-			(at 55.88 39.37 0)
+		(property "Footprint" "KH-TYPE-C-16P:KINGHELM_KH-TYPE-C-16P"
+			(at 63.5 34.29 0)
 			(effects
 				(font
 					(size 1.27 1.27)
 				)
+				(justify bottom)
 				(hide yes)
 			)
 		)
 		(property "Datasheet" ""
-			(at 55.88 39.37 0)
+			(at 63.5 34.29 0)
 			(effects
 				(font
@@
 		)
 		(property "Description" ""
-			(at 52.07 39.37 0)
+			(at 63.5 34.29 0)
 			(effects
 				(font
@@
 			)
 		)
-		(pin "4"
+		(property "MF" "kinghelm"
+			(at 63.5 34.29 0)
+			(effects
+				(font
+					(size 1.27 1.27)
+				)
+				(justify bottom)
+				(hide yes)
+			)
 		)
-		(pin "11"
+		(property "MAXIMUM_PACKAGE_HEIGHT" "3.41mm"
+			(at 63.5 34.29 0)
+			(effects
+				(font
+					(size 1.27 1.27)
+				)
+				(justify bottom)
+				(hide yes)
+			)
 		)
-		(pin "7"
+		(property "Package" "None"
+			(at 63.5 34.29 0)
+			(effects
+				(font
+					(size 1.27 1.27)
+				)
+				(justify bottom)
+				(hide yes)
+			)
 		)
-		(pin "3"
+		(property "Price" "None"
+			(at 63.5 34.29 0)
+			(effects
+				(font
+					(size 1.27 1.27)
+				)
+				(justify bottom)
+				(hide yes)
+			)
 		)
-		(pin "14"
+		(property "Check_prices" "https://www.snapeda.com/parts/KH-TYPE-C-16P/Kinghelm/view-part/?ref=eda"
+			(at 63.5 34.29 0)
+			(effects
+				(font
+					(size 1.27 1.27)
+				)
+				(justify bottom)
+				(hide yes)
+			)
 		)
-		(pin "6"
+		(property "STANDARD" "Manufacturer Recommendations"
+			(at 63.5 34.29 0)
+			(effects
+				(font
+					(size 1.27 1.27)
+				)
+				(justify bottom)
+				(hide yes)
+			)
 		)
-		(pin "8"
+		(property "PARTREV" "A0"
+			(at 63.5 34.29 0)
+			(effects
+				(font
+					(size 1.27 1.27)
+				)
+				(justify bottom)
+				(hide yes)
+			)
 		)
-		(pin "10"
+		(property "SnapEDA_Link" "https://www.snapeda.com/parts/KH-TYPE-C-16P/Kinghelm/view-part/?ref=snap"
+			(at 63.5 34.29 0)
+			(effects
+				(font
+					(size 1.27 1.27)
+				)
+				(justify bottom)
+				(hide yes)
+			)
 		)
-		(pin "5"
+		(property "MP" "KH-TYPE-C-16P"
+			(at 63.5 34.29 0)
+			(effects
+				(font
+					(size 1.27 1.27)
+				)
+				(justify bottom)
+				(hide yes)
+			)
 		)
-		(pin "1"
+		(property "Description_1" ""
+			(at 63.5 34.29 0)
+			(effects
+				(font
+					(size 1.27 1.27)
+				)
+				(justify bottom)
+				(hide yes)
+			)
 		)
-		(pin "9"
+		(property "SNAPEDA_PN" "KH-TYPE-C-16P"
+			(at 63.5 34.29 0)
+			(effects
+				(font
+					(size 1.27 1.27)
+				)
+				(justify bottom)
+				(hide yes)
+			)
 		)
-		(pin "12"
+		(property "Availability" "Not in stock"
+			(at 63.5 34.29 0)
+			(effects
+				(font
+					(size 1.27 1.27)
+				)
+				(justify bottom)
+				(hide yes)
+			)
 		)
-		(pin "13"
+		(property "MANUFACTURER" "Kinghelm"
+			(at 63.5 34.29 0)
+			(effects
+				(font
+					(size 1.27 1.27)
+				)
+				(justify bottom)
+				(hide yes)
+			)
 		)
-		(pin "2"
+		(pin "B6"
+		)
+		(pin "SH4"
+		)
+		(pin "B5"
+		)
+		(pin "A8"
+		)
+		(pin "SH3"
+		)
+		(pin "A5"
+		)
+		(pin "A1_B12"
+		)
+		(pin "A4_B9"
+		)
+		(pin "SH1"
+		)
+		(pin "A7"
+		)
+		(pin "A6"
+		)
+		(pin "A12_B1"
+		)
+		(pin "B8"
+		)
+		(pin "B7"
+		)
+		(pin "A9_B4"
+		)
+		(pin "SH2"
 		)
 		(instances

Commit message: updt
Parts:
- removed J1: ~, Connector_PinSocket_2.54mm:PinSocket_1x02_P2.54mm_Vertical, symbol _symbolsslime:POGO-F-2.5_1x2
- added VD1: 220k, Resistor_SMD:R_0603_1608Metric, symbol Device:R
- added VD2: 100k, Resistor_SMD:R_0603_1608Metric, symbol Device:R
- J2: footprint KH-TYPE-C-16P:KINGHELM_KH-TYPE-C-16P -> SlimeFootprints:KINGHELM_KH-TYPE-C-16P
Connections:
- net +5V: now also J2.A4_B9 (VBUS), J2.A9_B4 (VBUS)
- net ADC: now also VD1.1, VD2.2
- net BTS: now also VD1.2
- net DN: now also J2.A7 (DN1), J2.B7 (DN2)
- net DP: now also J2.A6 (DP1), J2.B6 (DP2)
- net GND: now also J2.A12_B1 (GND), J2.A1_B12 (GND), J2.SH1 (SHIELD), J2.SH2 (SHIELD), J2.SH3 (SHIELD), J2.SH4 (SHIELD), VD2.1
- net at R1.1: now also J2.B5 (CC2)
- net at R2.1: now also J2.A5 (CC1)
- no-connect marks 23 -> 24
Other:
- moved on the sheet: R1, R2
